Commit message: progress, yet no progress

File: source/isaaclab_sensor_learning/isaaclab_sensor_learning/urdf/linear_slider/linear_slider.urdf (robot description, URDF)
Before this commit: robot linear_slider, 6 links, 5 joints
Links:
- removed link base
- removed link base_link
- removed link flange
- removed link moving_base
- removed link tool0
- removed link world
- added link linear_slider__base_link, mass 20.0; collision box size=1.0 0.3 0.10; visual mesh filename=file:///home/luke/IsaacLab/source/isaaclab-sensor-learning/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 scale=0.001 0.001 0.001
- added link linear_slider__flange
- added link linear_slider__moving_base, mass 10.0; collision box size=0.22 0.202 0.118; visual mesh filename=file:///home/luke/IsaacLab/source/isaaclab-sensor-learning/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 scale=0.001 0.001 0.001
- added link linear_slider__tool0
Joints:
- removed joint base_joint
- removed joint base_link--base_joint
- removed joint flange--tool0_joint
- removed joint joint1
- removed joint moving_base--flange_joint
- added joint linear_slider__flange__tool0_joint: type fixed, parent linear_slider__flange, child linear_slider__tool0, origin xyz=0 0 0 rpy=0 0 0
- added joint linear_slider__joint1: type prismatic, parent linear_slider__base_link, child linear_slider__moving_base, origin xyz=0 0 0 rpy=0 0 0, axis 1 0 0, limit lower=-0.4 upper=0.4 effort=10 velocity=0.25
- added joint linear_slider__moving_base__flange_joint: type fixed, parent linear_slider__moving_base, child linear_slider__flange, origin xyz=0 0 0.05 rpy=0 0 0
